File: Kicad_Bloques/PLC/Digital.kicad_sch (KiCad schematic)
At the start: 0 parts

Commit message: Actualizacion Bloques e Investigacion
Parts:
- added C5: 0.1uf, symbol Device:C
- added D3: LED, symbol Device:LED
- added R2: 10k, symbol Device:R
- added R3: 2.2k, symbol Device:R
- added U4: Optocoupler_DC_PhotoNPN_AKEC, symbol Isolator:Optocoupler_DC_PhotoNPN_AKEC
Connections:
- new net: C5.1, R3.2, U4.1
- new net: C5.2, D3.2 (A), U4.2
- new net 3.3v: U4.4
- new net Digital_S1: R3.1
- new net GND: D3.1 (K), R2.2
- new net Out_D1: R2.1, U4.3
Other:
- note added: "Digital Block"
