File: Kicad_Bloques/PLC/Fuente.kicad_sch (KiCad schematic)
At the start: 0 parts

Commit message: Actualizacion bloques 9/2/2026{
Parts:
- added 24v1: Conn_01x02_Pin, Connector_Phoenix_GMSTB:PhoenixContact_GMSTBA_2,5_2-G-7,62_1x02_P7.62mm_Horizontal, symbol Connector:Conn_01x02_Pin
- added C1: 220nF, Capacitor_SMD:C_0805_2012Metric, symbol Device:C
- added C2: 100nF, symbol Device:C
- added C3: 330nF, Capacitor_SMD:C_0805_2012Metric, symbol Device:C
- added C4: 100nF, Capacitor_SMD:C_0805_2012Metric, symbol Device:C
- added D2: ABS2, Diode_SMD:Diode_Bridge_Diotec_ABS, symbol Diode_Bridge:ABS2
- added U2: LM7805_TO220, Package_TO_SOT_THT:TO-220-3_Vertical, symbol Regulator_Linear:LM7805_TO220
- added U3: LM7812_TO220, Package_TO_SOT_THT:TO-220-3_Vertical, symbol Regulator_Linear:LM7812_TO220
Connections:
- new net: 24v1.1 (Pin_1), D2.4
- new net: 24v1.2 (Pin_2), D2.3
- new net 12v: C4.1, U3.3 (VO)
- new net 24v: C1.1, C3.1, D2.1 (+), U2.1 (VI), U3.1 (VI)
- new net 5v: C2.1, U2.3 (VO)
- new net GND: C1.2, C2.2, C3.2, C4.2, D2.2 (-), U2.2 (GND), U3.2 (GND)
Other:
- note added: "12v regulator"
- note added: "24v Input"
- note added: "5v regulator"

Commit message: Actualizacion Bloques e Investigacion
Parts:
- added C6: 0.1uF, Capacitor_SMD:C_0805_2012Metric, symbol Device:C
- added C7: 0.1uF, symbol Device:C
- added C8, C9: 10uF, symbol Device:C
- added U6: AMS1117-3.3, Package_TO_SOT_SMD:SOT-223-3_TabPin2, symbol Regulator_Linear:AMS1117-3.3
Connections:
- net 5v: now also C6.1, C9.1, U6.3 (VI)
- net GND: now also C6.2, C7.2, C8.2, C9.2, U6.1 (GND)
- new net 3.3v: C7.1, C8.1, U6.2 (VO)
Other:
- note added: "3.3v regulator"
- moved on the sheet: C1, C2, C3, C4, U2, U3
