File: Kicad_Bloques/PLC/4-20mA.kicad_sch (KiCad schematic)
At the start: 0 parts

Commit message: Actualizacion bloque 4-20mA
Parts:
- added C12: 0.1uF, symbol Device:C
- added R8: 150R, symbol Device:R
- added R9: 100R, symbol Device:R
- added U5: MCP6002-xMC, Package_DFN_QFN:DFN-8-1EP_3x2mm_P0.5mm_EP1.75x1.45mm, symbol Amplifier_Operational:MCP6002-xMC
Connections:
- new net: R9.1, U5.1, U5.2 (-)
- new net +: C12.1, R8.1, U5.3 (+)
- new net -: U5.8 (V+)
- new net GND: C12.2, R8.2, U5.4 (V-), U5.9 (V-)
- new net Output_4-20mA: R9.2

Commit message: Actualizacion de bloques
Other:
- note added: "4-20mA Input"
Changed lines of the file:
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@@
 	(generator_version "9.0")
 	(paper "A4")
+	(text "4-20mA Input"
+		(exclude_from_sim no)
+		(at 88.392 61.468 0)
+		(effects
+			(font
+				(size 1.905 1.905)
+				(thickness 0.381)
+				(bold yes)
+			)
+		)
+	)
 	(junction
 		(at 113.03 72.39)
@@
 		)
 	)
+	(rule_area
+		(polyline
+			(pts
+				(xy 171.45 54.61) (xy 68.58 54.61) (xy 68.58 96.52) (xy 171.45 96.52)
+			)
+			(stroke
+				(width 0)
+				(type dash)
+			)
+			(fill
+				(type none)
+			)
+		)
+	)
