File: Kicad_Bloques/PLC/Relay.kicad_sch (KiCad schematic)
At the start: 0 parts

Commit message: Actualizacion bloques 9/2/2026{
Parts:
- added D1: 1N4148WT, Diode_SMD:D_SOD-523, symbol Diode:1N4148WT
- added K1: FINDER-34.51, Relay_THT:Relay_SPDT_Finder_34.51_Vertical, symbol Relay:FINDER-34.51
- added Q1: 2N3904, Package_TO_SOT_THT:TO-92_Inline, symbol Transistor_BJT:2N3904
- added R1: R, symbol Device:R
Connections:
- new net: Q1.2 (B), R1.2
- new net: D1.2 (A), K1.A2, Q1.3 (C)
- new net 24V: K1.11
- new net 5v: D1.1 (K), K1.A1
- new net GND: Q1.1 (E)
- new net Out_R_NC: K1.12
- new net Out_R_NO: K1.14
- new net R_Signal1: R1.1
Other:
- note added: "Relay Block"

Commit message: Actualizacion Bloques e Investigacion
Parts:
- added D4: LED, LED_SMD:LED_0805_2012Metric, symbol Device:LED
- added J6: Screw_Terminal_01x02, TerminalBlock:TerminalBlock_bornier-2_P5.08mm, symbol Connector:Screw_Terminal_01x02
- added R14: 470, Resistor_SMD:R_0805_2012Metric, symbol Device:R_Small
- added U7: ULN2003, Package_SO:SO-16_3.9x9.9mm_P1.27mm, symbol Transistor_Array:ULN2003
Connections:
- net 5v: now also R14.1
- net at D1.2 (A), K1.A2, Q1.3 (C): now also D4.1 (K)
- net 24V: no longer names the net of K1.11
- net 24V: now also J6.2 (Pin_2)
- net Out_R_NC: no longer names the net of K1.12
- net Out_R_NO: no longer names the net of K1.14
- net Out_R_NO: now also J6.1 (Pin_1)
- net R_Signal1 renamed Relay_S1
- net Relay_S1: now also U7.16 (O1)
- new net: D4.2 (A), R14.2
- new net Out_Relay: U7.1 (I1)
Other:
- moved on the sheet: R1

Commit message: Actualizacion de bloques
Parts:
- removed Q1: 2N3904, Package_TO_SOT_THT:TO-92_Inline, symbol Transistor_BJT:2N3904
- removed R1: R, symbol Device:R
Connections:
- net Relay_S1: now also D1.2 (A), D4.1 (K), K1.A2
Other:
- moved on the sheet: D4, J6, K1, R14, U7
