File: Tarea 3/Kicad_Bloques/PLC/Fuente.kicad_sch (KiCad schematic)
At the start: 13 parts, among them U2 LM7805_TO220, U3 LM7812_TO220, U6 AMS1117-3.3

Commit message: Organizando
Parts:
- removed D2: ABS2, Diode_SMD:Diode_Bridge_Diotec_ABS, symbol Diode_Bridge:ABS2
- added D2: SB120, Diode_THT:D_DO-41_SOD81_P10.16mm_Horizontal, symbol Diode:SB120
Connections:
- net 24v: now also D2.1 (K)
- net GND: now also 24v1.2 (Pin_2)
- net at 24v1.1 (Pin_1): now also D2.2 (A)
Changed lines of the file:
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@@
 	(wire
 		(pts
-			(xy 33.02 45.72) (xy 35.56 45.72)
+			(xy 33.02 45.72) (xy 40.64 45.72)
 		)
 		(stroke
@@
 	(wire
 		(pts
+			(xy 40.64 43.18) (xy 41.91 43.18)
+		)
+		(stroke
+			(width 0)
+			(type default)
+		)
+	)
+	(wire
+		(pts
 			(xy 200.66 54.61) (xy 207.01 54.61)
 		)
@@
 	(wire
 		(pts
-			(xy 35.56 43.18) (xy 35.56 36.83)
-		)
-		(stroke
-			(width 0)
-			(type default)
-		)
-	)
-	(wire
-		(pts
 			(xy 93.98 54.61) (xy 93.98 58.42)
 		)
@@
 	(wire
 		(pts
-			(xy 35.56 36.83) (xy 48.26 36.83)
-		)
-		(stroke
-			(width 0)
-			(type default)
-		)
-	)
-	(wire
-		(pts
-			(xy 33.02 43.18) (xy 35.56 43.18)
-		)
-		(stroke
-			(width 0)
-			(type default)
-		)
-	)
-	(wire
-		(pts
 			(xy 190.5 54.61) (xy 200.66 54.61)
 		)
@@
 	(wire
 		(pts
-			(xy 35.56 52.07) (xy 48.26 52.07)
-		)
-		(stroke
-			(width 0)
-			(type default)
-		)
-	)
-	(wire
-		(pts
 			(xy 198.12 44.45) (xy 200.66 44.45)
-		)
-		(stroke
-			(width 0)
-			(type default)
-		)
-	)
-	(wire
-		(pts
-			(xy 35.56 45.72) (xy 35.56 52.07)
 		)
 		(stroke
@@
 	(hierarchical_label "24v"
 		(shape output)
-		(at 55.88 44.45 0)
+		(at 41.91 43.18 0)
 		(effects
 			(font
@@
 	)
 	(symbol
+		(lib_id "Diode:SB120")
+		(at 36.83 43.18 180)
+		(unit 1)
+		(exclude_from_sim no)
+		(in_bom yes)
+		(on_board yes)
+		(dnp no)
+		(fields_autoplaced yes)
+		(property "Reference" "D2"
+			(at 37.1475 36.83 0)
+			(effects
+				(font
+					(size 1.27 1.27)
+				)
+			)
+		)
+		(property "Value" "SB120"
+			(at 37.1475 39.37 0)
+			(effects
+				(font
+					(size 1.27 1.27)
+				)
+			)
+		)
+		(property "Footprint" "Diode_THT:D_DO-41_SOD81_P10.16mm_Horizontal"
+			(at 36.83 38.735 0)
+			(effects
+				(font
+					(size 1.27 1.27)
+				)
+				(hide yes)
+			)
+		)
+		(property "Datasheet" "http://www.diodes.com/_files/datasheets/ds23022.pdf"
+			(at 36.83 43.18 0)
+			(effects
+				(font
+					(size 1.27 1.27)
+				)
+				(hide yes)
+			)
+		)
+		(property "Description" "20V 1A Schottky Barrier Rectifier Diode, DO-41"
+			(at 36.83 43.18 0)
+			(effects
+				(font
+					(size 1.27 1.27)
+				)
+				(hide yes)
+			)
+		)
+		(pin "1"
+		)
+		(pin "2"
+		)
+		(instances
+			(project ""
+				(path "/0c134be8-0195-4dcb-8651-b565a497cc9a/27cd8fbd-b108-47b8-ac4c-6fc7885b5b3e"
+					(reference "D2")
+					(unit 1)
+				)
+			)
+		)
+	)
+	(symbol
 		(lib_id "Device:C")
 		(at 104.14 50.8 0)
@@
 	)
 	(symbol
-		(lib_id "Diode_Bridge:ABS2")
-		(at 48.26 44.45 0)
-		(unit 1)
-		(exclude_from_sim no)
-		(in_bom yes)
-		(on_board yes)
-		(dnp no)
-		(property "Reference" "D2"
-			(at 48.514 44.196 0)
-			(effects
-				(font
-					(size 1.27 1.27)
-				)
-			)
-		)
-		(property "Value" "ABS2"
-			(at 48.26 44.958 0)
-			(effects
-				(font
-					(size 1.27 1.27)
-				)
-				(hide yes)
-			)
-		)
-		(property "Footprint" "Diode_SMD:Diode_Bridge_Diotec_ABS"
-			(at 52.07 41.275 0)
-			(effects
-				(font
-					(size 1.27 1.27)
-				)
-				(justify left)
-				(hide yes)
-			)
-		)
-		(property "Datasheet" "https://diotec.com/tl_files/diotec/files/pdf/datasheets/abs2.pdf"
-			(at 48.26 44.45 0)
-			(effects
-				(font
-					(size 1.27 1.27)
-				)
-				(hide yes)
-			)
-		)
-		(property "Description" "Miniature Glass Passivated Single-Phase Surface Mount Bridge Rectifiers, 140V Vrms, 0.8A If, ABS SMD package"
-			(at 48.26 44.45 0)
-			(effects
-				(font
-					(size 1.27 1.27)
-				)
-				(hide yes)
-			)
-		)
-		(pin "3"
-		)
-		(pin "1"
-		)
-		(pin "2"
-		)
-		(pin "4"
-		)
-		(instances
-			(project ""
-				(path "/0c134be8-0195-4dcb-8651-b565a497cc9a/27cd8fbd-b108-47b8-ac4c-6fc7885b5b3e"
-					(reference "D2")
-					(unit 1)
-				)
-			)
-		)
-	)
-	(symbol
 		(lib_id "power:GND")
-		(at 40.64 44.45 270)
+		(at 40.64 45.72 90)
 		(unit 1)
 		(exclude_from_sim no)
@@
 		(fields_autoplaced yes)
 		(property "Reference" "#PWR02"
-			(at 34.29 44.45 0)
+			(at 46.99 45.72 0)
 			(effects
 				(font
@@
 		)
 		(property "Value" "GND"
-			(at 39.37 40.64 90)
-			(effects
-				(font
-					(size 1.27 1.27)
-				)
+			(at 44.45 45.7199 90)
+			(effects
+				(font
+					(size 1.27 1.27)
+				)
+				(justify right)
 			)
 		)
 		(property "Footprint" ""
-			(at 40.64 44.45 0)
+			(at 40.64 45.72 0)
 			(effects
 				(font
@@
 		)
 		(property "Datasheet" ""
-			(at 40.64 44.45 0)
+			(at 40.64 45.72 0)
 			(effects
 				(font
@@
 		)
 		(property "Description" "Power symbol creates a global label with name \"GND\" , ground"
-			(at 40.64 44.45 0)
-			(effects
-				(font
+			(at 40.64 45.72 0)
+			(effects
+				(font
